Commit message: removed inertia from sensors for vertical liftoff

File: hector_models/hector_sensors_description/urdf/asus_camera.urdf.xacro (robot description, xacro)
@@ -13,9 +13,9 @@
       </joint>
       <link name="${name}_link">
-        <inertial>
+        <!-- <inertial>
           <mass value="0.200" />
           <origin xyz="0 0 0" rpy="0 0 0" />
           <inertia ixx="5.8083e-4" ixy="0" ixz="0" iyy="3.0833e-5" iyz="0" izz="5.9083e-4" />
-        </inertial>
+        </inertial> -->
         <visual>
           <origin xyz="0 0 0" rpy="0 0 0" />

File: hector_models/hector_sensors_description/urdf/hokuyo_utm30lx.urdf.xacro (robot description, xacro)
@@ -9,9 +9,9 @@
       </joint>
       <link name="${name}_frame">
-        <inertial>
+        <!-- <inertial>
           <mass value="0.270" />
           <origin xyz="0 0 0" rpy="0 0 0" />
           <inertia ixx="2.632e-4" ixy="0" ixz="0" iyy="2.632e-4" iyz="0" izz="1.62e-4" />
-        </inertial>
+        </inertial> -->
         <visual>
           <origin xyz="0 0 0" rpy="0 0 0" />
